File: csi.kicad_sch (KiCad schematic)
At the start: 65 parts, among them J7 Conn_FFC_WE_68715014522, J8 Conn_FFC_WE_68715014522, U24 AP22615A_TSOT26, U25 AP22615A_TSOT26, U26 PI4MSD5V9548AZDEX, U27 AP22615A_TSOT26, U28 AP22615A_TSOT26, U31 NTS0102_XSON, U32 NTS0102_XSON

Commit message: Complete baseboard routing, safety verification, and rename to Quadro
Parts:
- C100, C101, C42, C43, C89, C90, C91, C94, C95, C96, C97, C98, C99, D18, D20, D24, D25, J7, J8, R10, R103, R107, R108, R122, R132, R133, R161, R162, R163, R166, R167, R168, R171, R174, R179, R180, R193, R194, R197, R206, R36, R48, R50, R51, R6, R66, R67, R7, R8, R9, TP36, TP37, TP38, TP39, TP40, TP41, TP42, TP43, U24, U25, U26, U27, U28, U31, U32: Author Antmicro -> Quadro
Other:
- company: Antmicro Ltd -> Quadro
