File: jetson-orin-baseboard.kicad_pcb (KiCad board)
At the start: 8 copper layers, 120 x 60 mm, 681 parts, among them J1 Bus_M.2_2199230-6, J10 Molex_PicoBlade_1x4_0533980471, J11 Socket_Samtec_ERF8_2x40_ERF8-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, J12 Molex_Nano-Fit_1x2_SMD_105430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, J13 HDMI-Mini-C_WE_685119136923, J14 JST_SH_1x4_SM04B-SRSS-TB-LF-SN, J15 Bus_DDR4_SODIMM_CUSTOM_Jetson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, J2 Bus_M.2_1-2199230-6, J3 USB-C_GCT_USB4105-GF-A, J4 USB-C_WE_632723300011, J5 USB-C_WE_632723300011, J6 Bus_RJ45_5-2337992-8, J7 Conn_FFC_WE_68715014522, J8 Conn_FFC_WE_68715014522, J9 Tag-Connect_TC2050-IDC-NL_2x5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, M1 Jetson-Orin-NX-Nano, M3 Mech_M2_2280_H2.5mm, Q1 PJE138K, Q10 PJE138K, Q11 PJE138K, Q12 PJE138K, Q13 BCM857BS-7-F, Q14 BCM857BS-7-F, Q15 SSM3J332R, Q16 SSM3J332R, Q17 PJE138K, Q18 SSM3J332R, Q19 PJE138K, Q2 PJE138K, Q20 PJE138K, Q21 PJE138K, Q22 PJE138K, Q3 PJE138K, Q4 PJE138K, Q5 PJE138K, Q6 SSM3J332R, Q7 PJE138K, Q8 PJE138K, Q9 PJE138K, SW1 SW_SPDT_PCM12SMTR, U1 SIC431AED-T1-GE3, U10 TUSB1046-DCIRNQ, U11 TPD4E05U06QDQARQ1, U12 AP22615A_TSOT26, U13 TPD4E05U06QDQARQ1, U14 TPD4E05U06QDQARQ1, U15 TPD4E05U06QDQARQ1, U16 TPD4E05U06QDQARQ1, U17 HD3SS3220RNH, U18 AP22615A_TSOT26, U19 TPD4E05U06QDQARQ1, U2 74LVC2G07_SOT457, U20 TPD4E05U06QDQARQ1, U21 TPD4E05U06QDQARQ1, U22 TPS2372-3RGWR, U23 ULS-12_5-D48N-C, U24 AP22615A_TSOT26, U25 AP22615A_TSOT26, U26 PI4MSD5V9548AZDEX, U27 AP22615A_TSOT26, U28 AP22615A_TSOT26, U29 TPS259474, U3 74LVC2G07_SOT457, U30 TPD4E05U06QDQARQ1, U31 NTS0102_XSON, U32 NTS0102_XSON, U33 NTS0102_XSON, U34 PCAL6408A_VQFN, U35 AP22653_DFN, U36 TS3DV642RUARQ1, U37 74LVC2G14_SOT457, U38 74LVC1G175_SOT457, U39 ACPL-217-500E, U4 NTS0102_XSON, U40 SIC431AED-T1-GE3, U41 NCP730BMT330_WSON, U42 TPS7A0518P_SOT23-5, U43 NTS0102_XSON, U44 TPD4E05U06QDQARQ1, U45 TPD4E05U06QDQARQ1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

Commit message: Complete baseboard routing, safety verification, and rename to Quadro
Parts:
- removed C107, C114: C_1u_0402, antmicro-footprints:C_0402_1005Metric
- removed D39, D40, D45, D46, D49, D50: TPD1E0B04_XDFN-2, antmicro-footprints:XDFN-2_1x0.60mm
- removed J11: Socket_Samtec_ERF8_2x40_ERF8-040-05.0-L-DV-K-TR, antmicro-footprints:Conn_Socket_Samtec_ERF8_2x40_ERF8-040-05.0-L-DV-K-TR
- removed R100, R101, R102, R54, R64: R_4x330R_0402_array, antmicro-footprints:R_Array_4x0402
- removed R120, R121: R_0R_0402, antmicro-footprints:R_0402_1005Metric
- removed R335, R336: R_470R_0402, antmicro-footprints:R_0402_1005Metric
- added C167: 4n7, C_0402_1005Metric, B.Cu at (159.0, 82.0)
- added C168: 100nF, C_0402_1005Metric, B.Cu at (154.4, 91.5)
- added C169: 100nF, C_0402_1005Metric, B.Cu at (151.5, 83.5)
- added C170: 10uF, C_0603_1608Metric, F.Cu at (154.5, 70.0)
- added C171: 10uF, C_0603_1608Metric, F.Cu at (154.5, 72.5)
- added C172: 100nF, C_0402_1005Metric, F.Cu at (155.0, 75.0)
- added C173: 100nF, C_0402_1005Metric, F.Cu at (160.0, 81.5)
- added C174: 100nF, C_0402_1005Metric, F.Cu at (155.0, 85.0)
- added C175: 100nF, C_0402_1005Metric, F.Cu at (160.0, 91.5)
- added C176: 100nF, C_0402_1005Metric, F.Cu at (155.0, 95.0)
- added C177: 100nF, C_0402_1005Metric, F.Cu at (160.0, 101.5)
- added C178: 100nF, C_0402_1005Metric, F.Cu at (155.0, 105.0)
- added C179: 100nF, C_0402_1005Metric, F.Cu at (160.0, 102.5)
- added D64: PESD2CANFD24V-T, SOT-23, B.Cu at (155.0, 79.5)
- added F1: 1.1A, Fuse_1812_4532Metric, F.Cu at (160.0, 71.5)
- added F2: 0.75A, Fuse_1206_3216Metric, F.Cu at (166.0, 71.5)
- added J16: JST_SH_1x4_SM04B-SRSS-TB-LF-SN, antmicro-footprints:Conn_JST_SH_1x4_SM04B-SRSS-TB-LF-SN, B.Cu at (155.0, 73.0)
- added J17: Conn_02x20_Odd_Even, PinHeader_2x20_P2.54mm_Vertical_SMD, F.Cu at (173.0, 98.8)
- added R337: 60R4, R_0402_1005Metric, B.Cu at (159.0, 79.0)
- added R338: 60R4, R_0402_1005Metric, B.Cu at (159.0, 80.5)
- added R340: 10k, R_0402_1005Metric, B.Cu at (159.0, 84.5)
- added R341: 10k, R_0402_1005Metric, F.Cu at (155.0, 79.0)
- added R342: 10k, R_0402_1005Metric, F.Cu at (155.0, 89.0)
- added R343: 10k, R_0402_1005Metric, F.Cu at (155.0, 99.0)
- added R344: 10k, R_0402_1005Metric, F.Cu at (155.0, 109.0)
- added U49: TCAN1044V-Q1, SOIC-8_3.9x4.9mm_P1.27mm, B.Cu at (155.0, 86.5)
- added U51: TXS0108EPW, TSSOP-20_4.4x6.5mm_P0.65mm, F.Cu at (160.0, 77.0)
- added U52: TXS0108EPW, TSSOP-20_4.4x6.5mm_P0.65mm, F.Cu at (160.0, 87.0)
- added U53: TXS0108EPW, TSSOP-20_4.4x6.5mm_P0.65mm, F.Cu at (160.0, 97.0)
- added U54: TXS0108EPW, TSSOP-20_4.4x6.5mm_P0.65mm, F.Cu at (160.0, 107.0)
- REF** (x2): value antmicro-logo_scaled_15mm -> quadro-logo_scaled_15mm
Routing:
- net FAN_PWM: track 40.7 -> 194.4 mm, vias 2 -> 9
- net +1V8: track 252.7 -> 342.8 mm, vias 11 -> 12
- net /Expansion/+3V3_EXP: track 0.00 -> 87.1 mm, vias 0 -> 6
- net +3V3: track 319.9 -> 404.2 mm, vias 65 -> 67
- net +5V: track 96.1 -> 178.3 mm, vias 35 -> 37
- net I2C1_SDA: track 162.5 -> 238.1 mm, vias 3 -> 4
- net I2C1_SCL: track 161.3 -> 236.5 mm, vias 3 -> 4
- net USER_BTN0: track 83.0 -> 152.5 mm, vias 3 -> 4
- net GPIO010: track 120.9 -> 186.1 mm, vias 4 -> 9
- net USER_BTN1: track 87.5 -> 146.6 mm, vias 3 -> 4
- net ~{SPI0_CS1}: track 78.2 -> 134.3 mm, vias 3 -> 5
- net USER_LED1: track 111.7 -> 167.0 mm, vias 3 -> 5
- net GPIO07: track 140.5 -> 194.4 mm, vias 5 -> 8
- net /CSI/CSI3_0_D1_P: track 51.4 -> 102.8 mm
- net /CSI/CSI3_0_D1_N: track 51.3 -> 102.6 mm
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Other:
- board size 120 x 60 mm -> 150.2 x 60 mm
- board text added: "quadro"
