File: jetson-orin-baseboard.kicad_pcb (KiCad board)
At the start: 8 copper layers, 150.2 x 60 mm, 693 parts, among them J1 Bus_M.2_2199230-6, J10 Molex_PicoBlade_1x4_0533980471, J12 Molex_Nano-Fit_1x2_SMD_105430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, J13 HDMI-Mini-C_WE_685119136923, J14 JST_SH_1x4_SM04B-SRSS-TB-LF-SN, J15 Bus_DDR4_SODIMM_CUSTOM_Jetson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, J16 JST_SH_1x4_SM04B-SRSS-TB-LF-SN, J17 Conn_02x20_Odd_Even, J2 Bus_M.2_1-2199230-6, J3 USB-C_GCT_USB4105-GF-A, J4 USB-C_WE_632723300011, J5 USB-C_WE_632723300011, J6 Bus_RJ45_5-2337992-8, J7 Conn_FFC_WE_68715014522, J8 Conn_FFC_WE_68715014522, J9 Tag-Connect_TC2050-IDC-NL_2x5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, M1 Jetson-Orin-NX-Nano, M3 Mech_M2_2280_H2.5mm, Q1 PJE138K, Q10 PJE138K, Q11 PJE138K, Q12 PJE138K, Q13 BCM857BS-7-F, Q14 BCM857BS-7-F, Q15 SSM3J332R, Q16 SSM3J332R, Q17 PJE138K, Q18 SSM3J332R, Q19 PJE138K, Q2 PJE138K, Q20 PJE138K, Q21 PJE138K, Q22 PJE138K, Q3 PJE138K, Q4 PJE138K, Q5 PJE138K, Q6 SSM3J332R, Q7 PJE138K, Q8 PJE138K, Q9 PJE138K, SW1 SW_SPDT_PCM12SMTR, U1 SIC431AED-T1-GE3, U10 TUSB1046-DCIRNQ, U11 TPD4E05U06QDQARQ1, U12 AP22615A_TSOT26, U13 TPD4E05U06QDQARQ1, U14 TPD4E05U06QDQARQ1, U15 TPD4E05U06QDQARQ1, U16 TPD4E05U06QDQARQ1, U17 HD3SS3220RNH, U18 AP22615A_TSOT26, U19 TPD4E05U06QDQARQ1, U2 74LVC2G07_SOT457, U20 TPD4E05U06QDQARQ1, U21 TPD4E05U06QDQARQ1, U22 TPS2372-3RGWR, U23 ULS-12_5-D48N-C, U24 AP22615A_TSOT26, U25 AP22615A_TSOT26, U26 PI4MSD5V9548AZDEX, U27 AP22615A_TSOT26, U28 AP22615A_TSOT26, U29 TPS259474, U3 74LVC2G07_SOT457, U30 TPD4E05U06QDQARQ1, U31 NTS0102_XSON, U32 NTS0102_XSON, U33 NTS0102_XSON, U34 PCAL6408A_VQFN, U35 AP22653_DFN, U36 TS3DV642RUARQ1, U37 74LVC2G14_SOT457, U38 74LVC1G175_SOT457, U39 ACPL-217-500E, U4 NTS0102_XSON, U40 SIC431AED-T1-GE3, U41 NCP730BMT330_WSON, U42 TPS7A0518P_SOT23-5, U43 NTS0102_XSON, U44 TPD4E05U06QDQARQ1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

Commit message: save
Routing:
- net +3V3: track 404.2 -> 309.6 mm, vias 67 -> 59
- net SPI1_MOSI: track 103.9 -> 79.8 mm, vias 2 -> 0
- net SPI1_MISO: track 104.1 -> 81.9 mm, vias 2 -> 1
- net GND: track 635.0 -> 613.3 mm
- net ~{SPI1_CS1}: track 103.5 -> 83.0 mm, vias 2 -> 0
- net /Peripherals/USB_CONN_P: track 16.6 -> 3.46 mm
- net SPIO_MOSI: track 95.3 -> 84.4 mm
- net /Peripherals/USB_CONN_N: track 16.6 -> 6.02 mm
- net SPIO_SCK: track 104.6 -> 95.4 mm
- net /Peripherals/USBSS2_TX_CONN_P: track 7.50 -> 0.07 mm
- net /Peripherals/USBSS2_TX_CONN_N: track 7.62 -> 0.48 mm
- net PCIE2_CLK_N: track 53.9 -> 47.4 mm
- net PCIE2_CLK_P: track 53.9 -> 47.5 mm
- net PCIE3_RST*: track 124.7 -> 119.6 mm
- net /Peripherals/PCIE2_TX1_CONN_N: track 4.63 -> 0.77 mm
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