File: jetson-orin-baseboard.kicad_sch (KiCad schematic)
At the start: 4 parts

Commit message: Complete baseboard routing, safety verification, and rename to Quadro
Parts:
- H3, H4, H5, H6: Author Antmicro -> Quadro
Other:
- added sheet CAN (can.kicad_sch)
- added sheet Expansion (expansion.kicad_sch)
- note added: "github.com/quadro/jetson-orin-baseboard"
- note removed: "github.com/antmicro/jetson-orin-baseboard"
- company: Antmicro Ltd -> Quadro
Changed lines of the file:
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@@
 		(date "2025-03-12")
 		(rev "1.3.4")
-		(company "Antmicro Ltd")
-		(comment 1 "www.antmicro.com")
+		(company "Quadro")
+		(comment 1 "www.quadro.com")
 	)
 	(junction
@@
 		)
 	)
-	(text "github.com/antmicro/jetson-orin-baseboard"
+	(text "github.com/quadro/jetson-orin-baseboard"
 		(exclude_from_sim no)
 		(at 14.605 31.115 0)
@@
 			)
 		)
-		(property "Author" "Antmicro"
+		(property "Author" "Quadro"
 			(at 375.92 245.11 0)
 			(effects
@@
 			)
 		)
-		(property "Author" "Antmicro"
+		(property "Author" "Quadro"
 			(at 383.54 236.22 0)
 			(effects
@@
 			)
 		)
-		(property "Author" "Antmicro"
+		(property "Author" "Quadro"
 			(at 383.54 248.92 0)
 			(effects
@@
 			)
 		)
-		(property "Author" "Antmicro"
+		(property "Author" "Quadro"
 			(at 383.54 242.57 0)
 			(effects
@@
 			)
 		)
-		(property "Author" "Antmicro"
+		(property "Author" "Quadro"
 			(at 383.54 255.27 0)
 			(effects
@@
 				)
 			)
+		)
+	)
+	(sheet
+		(at 203.2 228.6)
+		(size 12.7 12.7)
+		(fields_autoplaced yes)
+		(stroke
+			(width 0.1524)
+			(type solid)
+		)
+		(fill
+			(color 0 0 0 0.0000)
+		)
+		(property "Sheetname" "CAN"
+			(at 203.2 227.8884 0)
+			(effects
+				(font
+					(size 1.27 1.27)
+				)
+				(justify left bottom)
+			)
+		)
+		(property "Sheetfile" "can.kicad_sch"
+			(at 203.2 241.8846 0)
+			(effects
+				(font
+					(size 1.27 1.27)
+				)
+				(justify left top)
+			)
+		)
+		(instances
+			(project "jetson-orin-baseboard"
+				(path "/4b393452-b11e-416e-bc83-918ae3cab2f1"
+					(page "11")
+				)
+			)
+		)
+	)
+	(sheet
+		(at 139.7 254)
+		(size 12.7 12.7)
+		(fields_autoplaced yes)
+		(stroke
+			(width 0.1524)
+			(type solid)
+		)
+		(fill
+			(color 0 0 0 0.0000)
+		)
+		(property "Sheetname" "Expansion"
+			(at 139.7 253.2884 0)
+			(effects
+				(font
+					(size 1.27 1.27)
+				)
+				(justify left bottom)
+			)
+		)
+		(property "Sheetfile" "expansion.kicad_sch"
+			(at 139.7 267.2846 0)
+			(effects
+				(font
+					(size 1.27 1.27)
+				)
+				(justify left top)
+			)
+		)
+		(instances
+			(project "jetson-orin-baseboard"
+				(path "/4b393452-b11e-416e-bc83-918ae3cab2f1"
+					(page "12")
+				)
+			)
