File: m-2.kicad_sch (KiCad schematic)
At the start: 61 parts, among them J1 Bus_M.2_2199230-6, J2 Bus_M.2_1-2199230-6, M3 Mech_M2_2280_H2.5mm, U2 74LVC2G07_SOT457, U3 74LVC2G07_SOT457, Y1 Oscillator_32.768kHz_ECS_2520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

Commit message: Complete baseboard routing, safety verification, and rename to Quadro
Parts:
- A2, C10, C11, C12, C13, C14, C15, C16, C17, C18, C19, C20, C21, C22, C23, C24, C25, C7, C8, C9, D1, D51, D52, J1, J2, M3, R13, R14, R143, R15, R16, R17, R18, R186, R187, R19, R20, R21, R22, R27, R28, R29, R30, R31, R32, R37, R38, R39, R52, SP7, SP8, TP10, TP11, TP12, TP6, TP7, TP8, TP9, U2, U3, Y1: Author Antmicro -> Quadro
Other:
- company: Antmicro Ltd -> Quadro
