File: peripherals.kicad_sch (KiCad schematic)
At the start: 93 parts, among them J10 Molex_PicoBlade_1x4_0533980471, J11 Socket_Samtec_ERF8_2x40_ERF8-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, J14 JST_SH_1x4_SM04B-SRSS-TB-LF-SN, J9 Tag-Connect_TC2050-IDC-NL_2x5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, Q10 PJE138K, Q9 PJE138K, U30 TPD4E05U06QDQARQ1, U33 NTS0102_XSON, U34 PCAL6408A_VQFN, U35 AP22653_DFN

Commit message: Complete baseboard routing, safety verification, and rename to Quadro
Parts:
- C104, C105, C106, C107, C108, C109, C110, C111, C112, C113, C114, C115, C130, C44, C48, D16, D17, D19, D21, D22, D23, D26, D27, D39, D40, D41, D42, D43, D44, D45, D46, D47, D48, D49, D50, D54, D56, D57, D58, D59, D63, J10, J11, J14, J9, Q10, Q9, R100, R101, R102, R112, R120, R121, R134, R141, R189, R190, R191, R192, R195, R204, R215, R216, R217, R218, R219, R222, R223, R230, R231, R232, R233, R234, R235, R242, R247, R248, R25, R26, R335, R336, R53, R54, R55, R62, R63, R64, S2, S3, U30, U33, U34, U35: Author Antmicro -> Quadro
Other:
- note added: "pinout compatible with www.github.com/quadro/ftdi-toolkit"
- note removed: "pinout compatible with www.github.com/antmicro/ftdi-toolkit"
- company: Antmicro Ltd -> Quadro
