File: supply.kicad_sch (KiCad schematic)
At the start: 124 parts, among them J12 Molex_Nano-Fit_1x2_SMD_105430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, Q11 PJE138K, Q13 BCM857BS-7-F, Q14 BCM857BS-7-F, Q15 SSM3J332R, Q16 SSM3J332R, Q18 SSM3J332R, Q22 PJE138K, Q5 PJE138K, Q6 SSM3J332R, Q7 PJE138K, Q8 PJE138K, SW1 SW_SPDT_PCM12SMTR, U1 SIC431AED-T1-GE3, U29 TPS259474, U37 74LVC2G14_SOT457, U38 74LVC1G175_SOT457, U40 SIC431AED-T1-GE3, U41 NCP730BMT330_WSON, U42 TPS7A0518P_SOT23-5, U48 TPS259474

Commit message: Complete baseboard routing, safety verification, and rename to Quadro
Parts:
- C102, C103, C116, C117, C118, C119, C120, C121, C122, C123, C124, C125, C126, C127, C128, C129, C134, C137, C142, C150, C151, C152, C153, C154, C155, C156, C157, C160, C161, C5, C50, C6, C83, C93, D28, D29, D30, D31, D32, D33, D36, D37, D53, D60, D61, D62, J12, L1, L4, Q11, Q13, Q14, Q15, Q16, Q18, Q22, Q5, Q6, Q7, Q8, R159, R164, R165, R169, R170, R172, R173, R175, R176, R177, R178, R181, R182, R183, R188, R236, R237, R238, R239, R240, R249, R250, R251, R252, R253, R254, R255, R256, R257, R258, R259, R260, R261, R263, R264, R268, R269, R272, R273, R274, R275, R276, R283, R284, R285, R286, S4, S5, SW1, TP14, TP23, TP33, TP52, TP53, TP54, TP55, U1, U29, U37, U38, U40, U41, U42, U48: Author Antmicro -> Quadro
Other:
- company: Antmicro Ltd -> Quadro
