File: usb.kicad_sch (KiCad schematic)
At the start: 140 parts, among them J3 USB-C_GCT_USB4105-GF-A, J4 USB-C_WE_632723300011, Q20 PJE138K, Q21 PJE138K, U10 TUSB1046-DCIRNQ, U11 TPD4E05U06QDQARQ1, U12 AP22615A_TSOT26, U13 TPD4E05U06QDQARQ1, U14 TPD4E05U06QDQARQ1, U15 TPD4E05U06QDQARQ1, U16 TPD4E05U06QDQARQ1, U47 NTS0102_XSON, U5 FT230X_QFN, U6 TPS65988DHRSHR, U7 W25Q80DV_USON, U8 NCP730BMT330_WSON, U9 AP22615A_TSOT26

Commit message: Complete baseboard routing, safety verification, and rename to Quadro
Parts:
- C136, C140, C141, C143, C144, C145, C146, C147, C148, C149, C158, C159, C26, C27, C28, C29, C30, C31, C32, C33, C34, C35, C36, C37, C45, C49, C53, C54, C55, C56, C57, C58, C59, C60, C61, C62, C63, C64, C65, D2, D3, D35, D4, D5, D6, D7, D8, D9, J3, J4, Q20, Q21, R104, R105, R106, R109, R110, R111, R117, R127, R130, R131, R144, R158, R205, R207, R244, R246, R262, R267, R270, R271, R33, R41, R42, R43, R44, R45, R46, R56, R57, R58, R59, R65, R68, R69, R70, R71, R72, R73, R74, R75, R76, R77, R78, R79, R81, R82, R83, R84, R85, R86, R87, R88, R89, R90, R91, R92, R93, R94, R95, R96, R97, R98, R99, TP1, TP13, TP17, TP18, TP19, TP20, TP24, TP25, TP26, TP27, TP28, TP30, U10, U11, U12, U13, U14, U15, U16, U47, U5, U6, U7, U8, U9: Author Antmicro -> Quadro
Other:
- company: Antmicro Ltd -> Quadro
