File: usb3.kicad_sch (KiCad schematic)
At the start: 51 parts, among them J5 USB-C_WE_632723300011, Q19 PJE138K, Q4 PJE138K, U17 HD3SS3220RNH, U18 AP22615A_TSOT26, U19 TPD4E05U06QDQARQ1, U20 TPD4E05U06QDQARQ1, U21 TPD4E05U06QDQARQ1

Commit message: Complete baseboard routing, safety verification, and rename to Quadro
Parts:
- C66, C67, C68, C69, C70, C71, C72, C73, C74, C75, D10, D11, J5, Q19, Q4, R113, R114, R115, R116, R118, R119, R124, R125, R126, R128, R135, R136, R137, R138, R139, R140, R184, R200, R201, R202, R203, R23, R24, R245, R265, R266, R60, R61, TP29, TP31, TP32, U17, U18, U19, U20, U21: Author Antmicro -> Quadro
Other:
- company: Antmicro Ltd -> Quadro
